File: ESPpower.kicad_pcb (KiCad board)
At the start: 2 copper layers, 64.8 x 92 mm, 58 parts, among them CON1 +7 TO +20VDC, J1 RJ12, J2 Display, J3 Conn_01x02_Male, J4 Conn_01x02_Male, M1 ESP-12, P1 Program, Q1 AO3400, SW1 Reset, SW2 Program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

Commit message: Fix U4 part number to FM24C256 Fix U1 part to AP1117-3.3
Parts:
- U1: value AP1117 -> AP1117-3.3
- U4: value 24C512 -> FM24C256
Changed lines of the file:
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@@
       (effects (font (size 1 1) (thickness 0.15)))
     )
-    (fp_text value "24C512" (at 0 3.56) (layer "F.Fab")
+    (fp_text value "FM24C256" (at 0 3.56) (layer "F.Fab")
       (effects (font (size 1 1) (thickness 0.15)))
     )
@@
       (effects (font (size 1 1) (thickness 0.15)))
     )
-    (fp_text value "AP1117" (at 3.03 4.42) (layer "F.Fab")
-      (effects (font (size 1 1) (thickness 0.15)))
-    )
+    (fp_text value "AP1117-3.3" (at 3.03 4.42) (layer "F.Fab")
+      (effects (font (size 1 1) (thickness 0.15)))
+    )

Commit message: Saved with later KiCAD version.
Parts:
- moved R5 1.65 mm to (57.0, 92.7)
- moved J4 0.57 mm to (48.6, 22.4)
- moved J3 0.56 mm to (48.6, 26.0)
- moved R11 0.23 mm to (53.8, 94.0)
Routing:
- net Net-(R11-Pad2): track 3.19 -> 5.57 mm
- net GND: track 55.0 -> 57.4 mm, vias 33 -> 34
- net /SDA: track 77.1 -> 75.7 mm
- net Net-(J4-Pad2): track 1.86 -> 2.80 mm
